File: TR-Switch.kicad_pcb (KiCad board)
At the start: 2 copper layers, 76.1 x 48.6 mm, 22 parts, among them J1 Conn_Coaxial, J2 Conn_Coaxial, J3 Conn_Coaxial, J4 USB_A, J5 Conn_01x02_Socket, J6 Conn_01x02_Socket, J7 Conn_01x02_Socket, K1 HF3-03, Q1 2N7000, SW1 Push_Button

Commit message: -docu + comments -new layout
Parts:
- removed D4: LED, LED_THT:LED_D5.0mm
- removed J6, J7: Conn_01x02_Socket, Connector_PinHeader_2.54mm:PinHeader_1x02_P2.54mm_Vertical
- removed RV3, RV4: 10kOhm, Potentiometer_THT:Potentiometer_Bourns_3386C_Horizontal
- removed SW1: Push_Button, Button_Switch_THT:SW_PUSH_6mm
- added G1: LOGO, Wiesel:wiesel-logo-kicad-back-white, F.Cu at (226.6, 119.6)
- added G11: LOGO, Wiesel:wiesel-logo-kicad-back-white, B.Cu at (226.6, 119.6)
- added REF11: ESD-Logo_6.6x6mm_SilkScreen, Symbol:ESD-Logo_6.6x6mm_SilkScreen, B.Cu at (234.2, 121.7)
- added REF22: OSHW-Logo2_7.3x6mm_SilkScreen, Symbol:OSHW-Logo2_7.3x6mm_SilkScreen, B.Cu at (242.4, 122.4)
- added REF33: WEEE-Logo_4.2x6mm_SilkScreen, Symbol:WEEE-Logo_4.2x6mm_SilkScreen, B.Cu at (249.0, 122.0)
- added REF44: KiCad-Logo2_5mm_SilkScreen, Symbol:KiCad-Logo2_5mm_SilkScreen, B.Cu at (241.6, 114.4)
- D1: value LED -> 1N4001; footprint LED_THT:LED_D5.0mm -> PCM_Diode_THT_AKL:D_DO-41_SOD81_P7.62mm_Horizontal
- D3: value LED -> PWR
- J4: value USB_A -> Conn_01x02_Socket; footprint Connector_USB:USB_A_Receptacle_GCT_USB1046 -> Connector_PinSocket_2.54mm:PinSocket_1x02_P2.54mm_Vertical
- J5: value Conn_01x02_Socket -> 3.5mm_Stereo_SymSmall_0.05; footprint Connector_PinHeader_2.54mm:PinHeader_1x02_P2.54mm_Vertical -> KSJ:Jack_3.5mm_CUI_SJ1-3533NG_Horizontal-wodo
- Q1: value 2N7000 -> 2N3904; footprint Package_TO_SOT_THT:TO-92_Inline -> PCM_Package_TO_SOT_THT_AKL:TO-92_Inline_Wide_EBC
- RV1: value 10kOhm -> 50Ohm
- RV2: value 10kOhm -> 1kOhm
- moved RV2 107.9 mm to (211.7, 85.3), turned to 90 degrees
- moved J5 105.2 mm to (246.4, 57.2), turned to -90 degrees
- moved Q1 101.6 mm to (222.9, 107.4), turned to 90 degrees
- moved D3 82.2 mm to (217.9, 56.3), turned to 180 degrees
- moved D2 64.2 mm to (210.2, 105.1), turned to 90 degrees
- moved J3 52.7 mm to (246.6, 104.4), turned to 0 degrees
- moved J4 49.0 mm to (226.7, 56.5), turned to -90 degrees
- moved RV1 43.6 mm to (217.0, 104.6), turned to 180 degrees
- moved D1 39.8 mm to (222.2, 85.5)
- moved REF1 37.6 mm to (234.2, 121.7)
- moved REF3 36.6 mm to (249.0, 122.0)
- moved J1 35.6 mm to (246.5, 69.2), turned to 0 degrees
- moved REF2 31.6 mm to (242.4, 122.4)
- moved J2 30.5 mm to (246.5, 86.6), turned to 0 degrees
- moved K1 28.7 mm to (234.3, 88.5), turned to 0 degrees
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- renumbered REF** to REF1, REF** to REF2, REF** to REF3, REF** to REF4
Connections:
- D1 pad 1: GND -> +5V
- D2 pad 1: unconnected-(D2-K-Pad1) -> Net-(D1-A)
- D2 pad 2: unconnected-(D2-A-Pad2) -> Net-(D2-A)
- D3 pad 1: Net-(D3-K) -> GND
- D3 pad 2: Net-(D3-A) -> Net-(D2-A)
- J4 pad 1: +5V -> GND
- J4 pad 2: unconnected-(J4-D--Pad2) -> +5V
- J5 pad 1: GND -> Net-(J2-In)
- J5 pad 2: Net-(J5-Pin_2) -> GND
- K1 pad 11: GND -> Net-(D1-A)
- K1 pad 14: Net-(J3-In) -> Net-(J2-In)
- K1 pad 6: Net-(J2-In) -> Net-(J3-In)
- Q1 pad 2: Net-(J5-Pin_2) -> Net-(Q1-B)
- Q1 pad 3: Net-(D3-K) -> Net-(D1-A)
- RV1 pad 1: Net-(D1-A) -> Net-(Q1-B)
- RV1 pad 2: +5V -> Net-(J2-In)
- RV1 pad 3: +5V -> Net-(J2-In)
- RV2 pad 1: Net-(J5-Pin_2) -> Net-(D2-A)
Routing:
- net GND: track 14.6 -> 80.8 mm, vias 5 -> 15
- net Net-(J2-In): track 21.0 -> 85.4 mm
- net Net-(D2-A): track 0.00 -> 48.5 mm
- net Net-(D1-A): track 8.50 -> 51.5 mm
- net Net-(J1-In): track 9.11 -> 20.7 mm
- net Net-(J3-In): track 18.9 -> 30.4 mm
- net +5V: track 42.5 -> 48.6 mm
- net Net-(Q1-B): track 0.00 -> 6.03 mm
Other:
- board size 76.1 x 48.6 mm -> 50 x 75 mm
- board text added: "+5V|GND"
- board text added: "1 kOhm"
- board text added: "50 Ohm"
- board text added: "ANT"
- board text added: "HF3-03"
- board text added: "J4"
- board text added: "PTT"
- board text added: "PWR"
- board text added: "RX"
- board text added: "TR-Switch 0.11 (C) WodoWiesel 01/10/2024"
- board text added: "TX"
- board text added: "USB"
- board text removed: "TR-Switch (C) WodoWiesel 06/06/2024"
